Commit message: update every thing depend on robot name

File: gazebo/robot_arm_three.gazebo.xacro (robot description, xacro)
@@ -1,13 +1,8 @@
 <?xml version="1.0"?>
-<!--
-Copied and modified from ROS1 example -
-https://github.com/ros-simulation/gazebo_ros_demos/blob/kinetic-devel/rrbot_description/urdf/rrbot.gazebo
--->
 <robot xmlns:xacro="http://ros.org/wiki/xacro">
-  <xacro:macro name="rrbot_gazebo" params="prefix">
+  <xacro:macro name="robot_arm_three_gazebo" params="prefix">
     <!-- ros_control plugin -->
     <gazebo>
       <plugin filename="gz_ros2_control-system" name="gz_ros2_control::GazeboSimROS2ControlPlugin">
-        <!-- <parameters>$(find system_hss)/config/ros2_controllers_with_trajctory.yaml</parameters> -->
         <parameters>$(find robot_arm_three)/config/ros2_controllers.yaml</parameters>
         <control_period>0.001</control_period>

File: ros2_control/robot_arm_three.ros2_control.xacro (robot description, xacro)
@@ -1,5 +1,5 @@
 <?xml version="1.0"?>
 <robot xmlns:xacro="http://www.ros.org/wiki/xacro">
-  <xacro:macro name="rrbot_ros2_control" params="name prefix use_gazebo:=^|false">
+  <xacro:macro name="robot_arm_three_ros2_control" params="name prefix use_gazebo:=^|false">
     <ros2_control name="${name}" type="system">
   <hardware>
@@ -9,5 +9,4 @@
   </hardware>
   <joint name="First_axis_joint">
-    <!-- State (okuma) -->
     <state_interface name="position"/>
     <state_interface name="velocity">
@@ -15,6 +14,4 @@
     </state_interface>
     <command_interface name="velocity"/>
-    <!-- Command (yazma) - SADECE position -->
-    <!-- <command_interface name="position"/> -->
   </joint>
   <joint name="Second_axis_joint">

File: urdf/robot_arm_three.urdf (robot description, URDF)
Before this commit: robot robot_arm_three, 14 links, 13 joints
Links:
- link First_Mil_link: geometry collision mesh filename=package://robot_arm_three/meshes/First_Mil_link.STL; visual mesh filename=package://robot_arm_three/meshes/First_Mil_link.STL
- link First_axis_link: geometry collision mesh filename=package://robot_arm_three/meshes/First_axis_link.STL; visual mesh filename=package://robot_arm_three/meshes/First_axis_link.STL
- link Moving_base_Link: geometry collision mesh filename=package://robot_arm_three/meshes/Moving_base_Link.STL; visual mesh filename=package://robot_arm_three/meshes/Moving_base_Link.STL
- link Second_axis_link: geometry collision mesh filename=package://robot_arm_three/meshes/Second_axis_link.STL; visual mesh filename=package://robot_arm_three/meshes/Second_axis_link.STL
- link Second_fixing_axis_link: geometry collision mesh filename=package://robot_arm_three/meshes/Second_fixing_axis_link.STL; visual mesh filename=package://robot_arm_three/meshes/Second_fixing_axis_link.STL
- link Second_mil_link: geometry collision mesh filename=package://robot_arm_three/meshes/Second_mil_link.STL; visual mesh filename=package://robot_arm_three/meshes/Second_mil_link.STL
- link Third_axis_link: geometry collision mesh filename=package://robot_arm_three/meshes/Third_axis_link.STL; visual mesh filename=package://robot_arm_three/meshes/Third_axis_link.STL
- link Third_fixing_axis_link: geometry collision mesh filename=package://robot_arm_three/meshes/Third_fixing_axis_link.STL; visual mesh filename=package://robot_arm_three/meshes/Third_fixing_axis_link.STL
- link base_link: geometry collision mesh filename=package://robot_arm_three/meshes/base_link.STL; visual mesh filename=package://robot_arm_three/meshes/base_link.STL
- link camera_link: geometry collision mesh filename=package://robot_arm_three/meshes/camera_link.STL; visual mesh filename=package://robot_arm_three/meshes/camera_link.STL
- link gripper_base_link: geometry collision mesh filename=package://robot_arm_three/meshes/gripper_base_link.STL; visual mesh filename=package://robot_arm_three/meshes/gripper_base_link.STL
- link left_gripper_hand_link: geometry collision mesh filename=package://robot_arm_three/meshes/left_gripper_hand_link.STL; visual mesh filename=package://robot_arm_three/meshes/left_gripper_hand_link.STL
- link right_gripper_hand_link: geometry collision mesh filename=package://robot_arm_three/meshes/right_gripper_hand_link.STL; visual mesh filename=package://robot_arm_three/meshes/right_gripper_hand_link.STL

File: urdf/robot_arm_three.urdf.xacro (robot description, xacro)
@@ -27,5 +27,5 @@
       <geometry>
         <mesh
-          filename="file:///home/ros2/Desktop/ros_ws/src/robot_arm_three/meshes/base_link.STL" />
+          filename="package://robot_arm_three/meshes/base_link.STL" />
       </geometry>
       <material
@@ -41,5 +41,5 @@
       <geometry>
         <mesh
-          filename="file:///home/ros2/Desktop/ros_ws/src/robot_arm_three/meshes/base_link.STL" />
+          filename="package://robot_arm_three/meshes/base_link.STL" />
       </geometry>
     </collision>
@@ -67,5 +67,5 @@
       <geometry>
         <mesh
-          filename="file:///home/ros2/Desktop/ros_ws/src/robot_arm_three/meshes/Moving_base_Link.STL" />
+          filename="package://robot_arm_three/meshes/Moving_base_Link.STL" />
       </geometry>
       <material
@@ -81,5 +81,5 @@
       <geometry>
         <mesh
-          filename="file:///home/ros2/Desktop/ros_ws/src/robot_arm_three/meshes/Moving_base_Link.STL" />
+          filename="package://robot_arm_three/meshes/Moving_base_Link.STL" />
       </geometry>
     </collision>
@@ -120,5 +120,5 @@
       <geometry>
         <mesh
-          filename="file:///home/ros2/Desktop/ros_ws/src/robot_arm_three/meshes/First_axis_link.STL" />
+          filename="package://robot_arm_three/meshes/First_axis_link.STL" />
       </geometry>
       <material
@@ -134,5 +134,5 @@
       <geometry>
         <mesh
-          filename="file:///home/ros2/Desktop/ros_ws/src/robot_arm_three/meshes/First_axis_link.STL" />
+          filename="package://robot_arm_three/meshes/First_axis_link.STL" />
       </geometry>
     </collision>
@@ -186,5 +186,5 @@
       <geometry>
         <mesh
-          filename="file:///home/ros2/Desktop/ros_ws/src/robot_arm_three/meshes/First_Mil_link.STL" />
+          filename="package://robot_arm_three/meshes/First_Mil_link.STL" />
       </geometry>
       <material
@@ -200,5 +200,5 @@
       <geometry>
         <mesh
-          filename="file:///home/ros2/Desktop/ros_ws/src/robot_arm_three/meshes/First_Mil_link.STL" />
+          filename="package://robot_arm_three/meshes/First_Mil_link.STL" />
       </geometry>
     </collision>
@@ -239,5 +239,5 @@
       <geometry>
         <mesh
-          filename="file:///home/ros2/Desktop/ros_ws/src/robot_arm_three/meshes/Second_fixing_axis_link.STL" />
+          filename="package://robot_arm_three/meshes/Second_fixing_axis_link.STL" />
       </geometry>
       <material
@@ -253,5 +253,5 @@
       <geometry>
         <mesh
-          filename="file:///home/ros2/Desktop/ros_ws/src/robot_arm_three/meshes/Second_fixing_axis_link.STL" />
+          filename="package://robot_arm_three/meshes/Second_fixing_axis_link.STL" />
       </geometry>
     </collision>
@@ -292,5 +292,5 @@
       <geometry>
         <mesh
-          filename="file:///home/ros2/Desktop/ros_ws/src/robot_arm_three/meshes/Second_axis_link.STL" />
+          filename="package://robot_arm_three/meshes/Second_axis_link.STL" />
       </geometry>
       <material
@@ -306,5 +306,5 @@
       <geometry>
         <mesh
-          filename="file:///home/ros2/Desktop/ros_ws/src/robot_arm_three/meshes/Second_axis_link.STL" />
+          filename="package://robot_arm_three/meshes/Second_axis_link.STL" />
       </geometry>
     </collision>
@@ -358,5 +358,5 @@
       <geometry>
         <mesh
-          filename="file:///home/ros2/Desktop/ros_ws/src/robot_arm_three/meshes/Second_mil_link.STL" />
+          filename="package://robot_arm_three/meshes/Second_mil_link.STL" />
       </geometry>
       <material
@@ -372,5 +372,5 @@
       <geometry>
         <mesh
-          filename="file:///home/ros2/Desktop/ros_ws/src/robot_arm_three/meshes/Second_mil_link.STL" />
+          filename="package://robot_arm_three/meshes/Second_mil_link.STL" />
       </geometry>
     </collision>
@@ -411,5 +411,5 @@
       <geometry>
         <mesh
-          filename="file:///home/ros2/Desktop/ros_ws/src/robot_arm_three/meshes/Third_fixing_axis_link.STL" />
+          filename="package://robot_arm_three/meshes/Third_fixing_axis_link.STL" />
       </geometry>
       <material
@@ -425,5 +425,5 @@
       <geometry>
         <mesh
-          filename="file:///home/ros2/Desktop/ros_ws/src/robot_arm_three/meshes/Third_fixing_axis_link.STL" />
+          filename="package://robot_arm_three/meshes/Third_fixing_axis_link.STL" />
       </geometry>
     </collision>
@@ -464,5 +464,5 @@
       <geometry>
         <mesh
-          filename="file:///home/ros2/Desktop/ros_ws/src/robot_arm_three/meshes/Third_axis_link.STL" />
+          filename="package://robot_arm_three/meshes/Third_axis_link.STL" />
       </geometry>
       <material
@@ -478,5 +478,5 @@
       <geometry>
         <mesh
-          filename="file:///home/ros2/Desktop/ros_ws/src/robot_arm_three/meshes/Third_axis_link.STL" />
+          filename="package://robot_arm_three/meshes/Third_axis_link.STL" />
       </geometry>
     </collision>
@@ -530,5 +530,5 @@
       <geometry>
         <mesh
-          filename="file:///home/ros2/Desktop/ros_ws/src/robot_arm_three/meshes/camera_link.STL" />
+          filename="package://robot_arm_three/meshes/camera_link.STL" />
       </geometry>
       <material
@@ -544,5 +544,5 @@
       <geometry>
         <mesh
-          filename="file:///home/ros2/Desktop/ros_ws/src/robot_arm_three/meshes/camera_link.STL" />
+          filename="package://robot_arm_three/meshes/camera_link.STL" />
       </geometry>
     </collision>
@@ -613,5 +613,5 @@
       <geometry>
         <mesh
-          filename="file:///home/ros2/Desktop/ros_ws/src/robot_arm_three/meshes/gripper_base_link.STL" />
+          filename="package://robot_arm_three/meshes/gripper_base_link.STL" />
       </geometry>
       <material
@@ -627,5 +627,5 @@
       <geometry>
         <mesh
-          filename="file:///home/ros2/Desktop/ros_ws/src/robot_arm_three/meshes/gripper_base_link.STL" />
+          filename="package://robot_arm_three/meshes/gripper_base_link.STL" />
       </geometry>
     </collision>
@@ -666,5 +666,5 @@
       <geometry>
         <mesh
-          filename="file:///home/ros2/Desktop/ros_ws/src/robot_arm_three/meshes/right_gripper_hand_link.STL" />
+          filename="package://robot_arm_three/meshes/right_gripper_hand_link.STL" />
       </geometry>
       <material
@@ -680,5 +680,5 @@
       <geometry>
         <mesh
-          filename="file:///home/ros2/Desktop/ros_ws/src/robot_arm_three/meshes/right_gripper_hand_link.STL" />
+          filename="package://robot_arm_three/meshes/right_gripper_hand_link.STL" />
       </geometry>
     </collision>
@@ -729,5 +729,5 @@
       <geometry>
         <mesh
-          filename="file:///home/ros2/Desktop/ros_ws/src/robot_arm_three/meshes/left_gripper_hand_link.STL" />
+          filename="package://robot_arm_three/meshes/left_gripper_hand_link.STL" />
       </geometry>
       <material
@@ -743,5 +743,5 @@
       <geometry>
         <mesh
-          filename="file:///home/ros2/Desktop/ros_ws/src/robot_arm_three/meshes/left_gripper_hand_link.STL" />
+          filename="package://robot_arm_three/meshes/left_gripper_hand_link.STL" />
       </geometry>
     </collision>
